File: wordclock_pcb.sch (KiCad schematic (older format))
At the start: 33 parts, among them IC1 ATmega328P, J1 MYUSBCONN5, J2 Stecker 1, J3 Stecker 2, J4 Stecker 3, Q1 2N3904, Q2 2N3904, SW1 MYSWITCH2, SW2 MYSWITCH_reduced, SW3 MYSWITCH_reduced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

Commit message: Delete old pcb design and arrange footprints
Changed lines of the file:
@@
 EESchema Schematic File Version 4
 LIBS:wordclock_pcb-cache
-EELAYER 29 0
+EELAYER 30 0
 EELAYER END
 $Descr A4 11693 8268
@@
 L power:PWR_FLAG #FLG01
 U 1 1 5A023C8C
-P 700 750
-F 0 "#FLG01" H 700 825 50  0001 C CNN
-F 1 "PWR_FLAG" H 700 900 50  0000 C CNN
-F 2 "" H 700 750 50  0001 C CNN
-F 3 "" H 700 750 50  0001 C CNN
-	1    700  750
+P 1500 2200
+F 0 "#FLG01" H 1500 2275 50  0001 C CNN
+F 1 "PWR_FLAG" H 1500 2350 50  0000 C CNN
+F 2 "" H 1500 2200 50  0001 C CNN
+F 3 "" H 1500 2200 50  0001 C CNN
+	1    1500 2200
 	1    0    0    -1
 $EndComp
@@
 L power:PWR_FLAG #FLG03
 U 1 1 5A1B21C2
-P 1150 750
-F 0 "#FLG03" H 1150 825 50  0001 C CNN
-F 1 "PWR_FLAG" H 1150 900 50  0000 C CNN
-F 2 "" H 1150 750 50  0001 C CNN
-F 3 "" H 1150 750 50  0001 C CNN
-	1    1150 750
-	1    0    0    -1
-$EndComp
-$Comp
-L power:GND #PWR04
-U 1 1 5A1B22E2
-P 700 900
-F 0 "#PWR04" H 700 650 50  0001 C CNN
-F 1 "GND" H 700 750 50  0000 C CNN
-F 2 "" H 700 900 50  0001 C CNN
-F 3 "" H 700 900 50  0001 C CNN
-	1    700  900
+P 1650 1900
+F 0 "#FLG03" H 1650 1975 50  0001 C CNN
+F 1 "PWR_FLAG" H 1650 2050 50  0000 C CNN
+F 2 "" H 1650 1900 50  0001 C CNN
+F 3 "" H 1650 1900 50  0001 C CNN
+	1    1650 1900
 	1    0    0    -1
 $EndComp
@@
 $EndComp
 $Comp
-L power:+5V #PWR012
-U 1 1 5A2390CA
-P 1150 850
-F 0 "#PWR012" H 1150 700 50  0001 C CNN
-F 1 "+5V" H 1150 990 50  0000 C CNN
-F 2 "" H 1150 850 50  0001 C CNN
-F 3 "" H 1150 850 50  0001 C CNN
-	1    1150 850
-	-1   0    0    1
-$EndComp
-$Comp
 L power:+5V #PWR013
 U 1 1 5A239231
-P 1350 1850
-F 0 "#PWR013" H 1350 1700 50  0001 C CNN
-F 1 "+5V" H 1350 1990 50  0000 C CNN
-F 2 "" H 1350 1850 50  0001 C CNN
-F 3 "" H 1350 1850 50  0001 C CNN
-	1    1350 1850
+P 1350 1650
+F 0 "#PWR013" H 1350 1500 50  0001 C CNN
+F 1 "+5V" H 1350 1790 50  0000 C CNN
+F 2 "" H 1350 1650 50  0001 C CNN
+F 3 "" H 1350 1650 50  0001 C CNN
+	1    1350 1650
 	1    0    0    -1
 $EndComp
@@
 Connection ~ 4350 850
 Wire Wire Line
-	1150 750  1150 850
-Wire Wire Line
-	700  750  700  900
-Wire Wire Line
 	1100 1850 1350 1850
 Wire Wire Line
@@
 	1350 1850 1350 1900
 Wire Wire Line
-	1350 1900 1800 1900
+	1350 1900 1650 1900
 Connection ~ 1800 1900
 Connection ~ 2100 1900
 Connection ~ 2400 1900
 Wire Wire Line
-	1350 2200 1800 2200
+	1350 2200 1500 2200
 Wire Wire Line
 	1350 2250 1350 2200
@@
 Wire Wire Line
 	7200 2700 7200 2750
+Connection ~ 1650 1900
+Wire Wire Line
+	1650 1900 1800 1900
+Connection ~ 1500 2200
+Wire Wire Line
+	1500 2200 1800 2200
+Wire Wire Line
+	1350 1850 1350 1650
+Connection ~ 1350 1850
 $EndSCHEMATC
